File: neovibe/neovibe.kicad_sch (KiCad schematic)
At the start: 34 parts, among them J1 AudioJack2, J2 AudioJack2, Q1 2N3904, Q2 2N3904, Q3 2N3904, SW1 SW_Push_DPDT, SW2 SW_SPDT

Commit message: stuff
Parts:
- added C, F, G, H, I, J, K, O, X: Conn_01x01, symbol Connector_Generic:Conn_01x01
- added C10, C11, C13, C14, C17 (x2), C19, C20, C21, C6, C7, C8: 1uF 50V, symbol Device:C_Polarized
- added C12: 0.470pF, symbol Device:C
- added C15: 0.0047uF, symbol Device:C
- added C22, C23: 10uF 25V, symbol Device:C_Polarized
- added C24, C25: 1000uF 35V, symbol Device:C_Polarized
- added C26: C, symbol Device:C
- added C5: 0.015uF, symbol Device:C
- added C9: 0.22uF, symbol Device:C
- added D: D, symbol Connector_Generic:Conn_01x01
- added D1, D2: D, symbol Device:D
- added D3: DF01M, Diode_THT:Diode_Bridge_DIP-4_W7.62mm_P5.08mm, symbol Diode_Bridge:DF01M
- added E: E, symbol Connector_Generic:Conn_01x01
- added LA1: Lamp, symbol Device:Lamp
- added Q10, Q11, Q12, Q13, Q4, Q5, Q6, Q7, Q8, Q9: 2N3904, symbol Device:Q_NPN_BCE
- added R12, R20, R21, R24, R33: 47K, symbol Device:R
- added R13, R14, R19, R25, R26, R30, R32: 100K, symbol Device:R
- added R15, R16, R17, R18, R22, R23, R27, R28, R29, R31, R34, R41, R42, R43: 4.7K, symbol Device:R
- added R39: 3.3K, symbol Device:R
- added R40: 2.2M, symbol Device:R
- added R44, R45: 220K, symbol Device:R
- added R46, R47, R48, R49, R50: R, symbol Device:R
- added RV1: R_Potentiometer, symbol Device:R_Potentiometer
- added RV2: R_Potentiometer_Trim, symbol Device:R_Potentiometer_Trim
- added RV_Speed: 100K Rev Log, symbol Device:R_Potentiometer_Dual
- added R_LDR1, R_LDR2, R_LDR3, R_LDR4: LDR03, OptoDevice:R_LDR_10x8.5mm_P7.6mm_Vertical, symbol Sensor_Optical:LDR03
- added U1: L7815, symbol Regulator_Linear:L7815
- renumbered A to A1, B to B1, C to C16, L to L1, M to M1, N to N1, RV_Volume to RV_Volume1
Connections:
- net +15V: now also C26.1, Q10.2 (C), Q4.2 (C), Q6.2 (C), Q8.2 (C), R14.1, R18.1, R20.1, R22.1, R26.1, R29.1, R30.1, U1.1 (IN)
- net GND: now also C21.2, C24.2, C25.2, C26.2, D3.2 (-), F.1 (Pin_1), I.1 (Pin_1), O.1 (Pin_1), R12.2, R17.2, R21.2, R23.2, R24.2, R31.2, R33.2, R34.2, R41.2, R46.2, R50.1, RV1.3, RV2.2, RV2.3, U1.2 (GND)
- net at R36.2: now also R37.2, C17.2
- net at C18.1, Q3.3 (E), R9.1: now also C6.2
- net at Q3.2 (C), R11.2: now also C5.1
- new net: C12.1, Q7.2 (C), R22.2
- new net: C12.2, Q8.1 (B), R25.1, R27.1
- new net: C5.2, Q4.1 (B), R13.1, R15.1
- new net: C19.2, C20.1, D1.1 (K), D2.2 (A), R42.1, R44.1
- new net: C20.2, C21.1, D1.2 (A), D2.1 (K), R43.1, R45.1
- new net: C13.1, R30.2, R32.2, R33.1
- new net: C11.1, R_LDR4.2
- new net: C10.2, C11.2, Q7.3 (E), R23.1
- new net: C7.1, R12.1, R13.2, R14.2
- new net: C.1 (Pin_1), C22.1, Q12.3 (E), R44.2, R45.2, R46.1
- new net: C10.1, R19.2, R20.2, R21.1
- new net: R27.2, R_LDR4.1
- new net: C23.2, H.1 (Pin_1), RV1.2
- new net: C15.2, Q10.1 (B), R28.1, R32.1
- new net: C17.1, R24.1, R25.2, R26.2
- new net: C22.2, G.1 (Pin_1), RV1.1
- new net: R39.1, R40.1, R41.1
- new net: C9.1, Q5.2 (C), R18.2
- new net: C9.2, Q6.1 (B), R16.1, R19.1
- new net: Q8.3 (E), Q9.1 (B)
- new net: C13.2, C17.1, Q10.3 (E), R34.1
- new net: C23.1, R49.1
- new net: Q13.1 (B), R47.1, R49.2, R50.2, X.1 (Pin_1)
- new net: R48.1, RV2.1
- new net: Q6.3 (E), Q7.1 (B)
- new net: C24.1, C25.1, D3.1 (+), LA1.2 (+), Q11.2 (C), Q12.2 (C), Q13.2 (C), R39.2, R47.2, U1.3 (OUT)
- new net: Q4.3 (E), Q5.1 (B)
- new net: C7.2, C8.2, Q5.3 (E), R17.1
- new net: C19.1, Q11.1 (B), R40.2
- new net: Q11.3 (E), Q12.1 (B)
- new net: R16.2, R_LDR2.1
- new net: C8.1, R_LDR2.2
- new net: C15.1, Q9.2 (C), R29.2
- new net: D3.4, J.1 (Pin_1)
- new net: E.1 (Pin_1), R43.2
- new net: C6.1, R_LDR1.2
- new net: C14.2, C17.2, Q9.3 (E), R31.1
- new net: Q13.3 (E), R48.2
- new net: D3.3, K.1 (Pin_1)
- new net: C14.1, R_LDR3.2
- new net: R15.2, R_LDR1.1
- new net: D.1 (Pin_1), R42.2
- new net: R28.2, R_LDR3.1
- new net: RV_Speed.2, RV_Speed.3
- new net: RV_Speed.5, RV_Speed.6

Commit message: fix ec
Parts:
- Connector_C: renamed from C; value Conn_01x01 -> C_connector
- renumbered C13 to C100, C17 to C13
Connections:
- net GND: now also C3.2
- net at R7.2: now also Q1.2 (C), Q2.1 (B)
- net at C24.1, C25.1, D3.1 (+)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: no longer Q13.2 (C), R47.2
- net at E.1 (Pin_1), R43.2: now also RV_Speed.1
- net at C2.1, R4.1, R6.1: now also Q2.3 (E)
- net at D.1 (Pin_1), R42.2: now also RV_Speed.4
- net at LA1.1 (-): now also Q13.2 (C), R47.2
Changed lines of the file:
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@@
   (junction (at 119.38 82.55) (diameter 0) (color 0 0 0 0)
   )
+  (junction (at 45.72 201.93) (diameter 0) (color 0 0 0 0)
+  )
   (junction (at 165.1 187.96) (diameter 0) (color 0 0 0 0)
   )
@@
   (junction (at 40.64 176.53) (diameter 0) (color 0 0 0 0)
   )
-  (junction (at 151.13 154.94) (diameter 0) (color 0 0 0 0)
-  )
   (junction (at 176.53 179.07) (diameter 0) (color 0 0 0 0)
   )
@@
   (junction (at 148.59 45.72) (diameter 0) (color 0 0 0 0)
   )
+  (junction (at 151.13 166.37) (diameter 0) (color 0 0 0 0)
+  )
   (junction (at 160.02 35.56) (diameter 0) (color 0 0 0 0)
   )
@@
   (junction (at 30.48 185.42) (diameter 0) (color 0 0 0 0)
   )
+  (junction (at 85.09 50.8) (diameter 0) (color 0 0 0 0)
+  )
   (junction (at 45.72 44.45) (diameter 0) (color 0 0 0 0)
   )
@@
   (junction (at 111.76 154.94) (diameter 0) (color 0 0 0 0)
   )
-  (junction (at 151.13 166.37) (diameter 0) (color 0 0 0 0)
+  (junction (at 80.01 34.29) (diameter 0) (color 0 0 0 0)
+  )
+  (junction (at 52.07 201.93) (diameter 0) (color 0 0 0 0)
   )
   (junction (at 236.22 113.03) (diameter 0) (color 0 0 0 0)
@@
     (stroke (width 0) (type default))
   )
+  (wire (pts (xy 52.07 201.93) (xy 57.15 201.93))
+    (stroke (width 0) (type default))
+  )
   (wire (pts (xy 45.72 52.07) (xy 45.72 63.5))
     (stroke (width 0) (type default))
@@
     (stroke (width 0) (type default))
   )
+  (wire (pts (xy 80.01 34.29) (xy 80.01 35.56))
+    (stroke (width 0) (type default))
+  )
   (wire (pts (xy 130.81 172.72) (xy 130.81 200.66))
     (stroke (width 0) (type default))
@@
     (stroke (width 0) (type default))
   )
-  (wire (pts (xy 59.69 223.52) (xy 52.07 223.52))
-    (stroke (width 0) (type default))
-  )
   (wire (pts (xy 38.1 55.88) (xy 38.1 63.5))
     (stroke (width 0) (type default))
@@
     (stroke (width 0) (type default))
   )
+  (wire (pts (xy 85.09 50.8) (xy 87.63 50.8))
+    (stroke (width 0) (type default))
+  )
   (wire (pts (xy 16.51 199.39) (xy 29.21 199.39))
     (stroke (width 0) (type default))
@@
     (stroke (width 0) (type default))
   )
-  (wire (pts (xy 111.76 154.94) (xy 151.13 154.94))
+  (wire (pts (xy 111.76 154.94) (xy 176.53 154.94))
     (stroke (width 0) (type default))
   )
@@
     (stroke (width 0) (type default))
   )
-  (wire (pts (xy 151.13 154.94) (xy 176.53 154.94))
-    (stroke (width 0) (type default))
-  )
   (wire (pts (xy 96.52 210.82) (xy 100.33 210.82))
     (stroke (width 0) (type default))
@@
     (stroke (width 0) (type default))
   )
+  (wire (pts (xy 87.63 35.56) (xy 87.63 50.8))
+    (stroke (width 0) (type default))
+  )
   (wire (pts (xy 81.28 187.96) (xy 81.28 189.23))
     (stroke (width 0) (type default))
@@
     (stroke (width 0) (type default))
   )
-  (wire (pts (xy 57.15 203.2) (xy 57.15 213.36))
+  (wire (pts (xy 57.15 201.93) (xy 57.15 213.36))
     (stroke (width 0) (type default))
   )
@@
     (stroke (width 0) (type default))
   )
-  (wire (pts (xy 52.07 203.2) (xy 57.15 203.2))
-    (stroke (width 0) (type default))
-  )
   (wire (pts (xy 125.73 0) (xy 123.19 0))
     (stroke (width 0) (type default))
@@
     (stroke (width 0) (type default))
   )
+  (wire (pts (xy 52.07 223.52) (xy 59.69 223.52))
+    (stroke (width 0) (type default))
+  )
   (wire (pts (xy 143.51 45.72) (xy 148.59 45.72))
     (stroke (width 0) (type default))
@@
     (stroke (width 0) (type default))
   )
+  (wire (pts (xy 121.92 148.59) (xy 151.13 148.59))
+    (stroke (width 0) (type default))
+  )
   (wire (pts (xy 31.75 31.75) (xy 31.75 55.88))
     (stroke (width 0) (type default))
@@
     (stroke (width 0) (type default))
   )
+  (wire (pts (xy 59.69 38.1) (xy 59.69 39.37))
+    (stroke (width 0) (type default))
+  )
   (wire (pts (xy 43.18 81.28) (xy 58.42 81.28))
     (stroke (width 0) (type default))
@@
     (stroke (width 0) (type default))
   )
-  (wire (pts (xy 151.13 154.94) (xy 151.13 166.37))
-    (stroke (width 0) (type default))
-  )
-  (wire (pts (xy 45.72 203.2) (xy 45.72 204.47))
+  (wire (pts (xy 45.72 201.93) (xy 45.72 204.47))
     (stroke (width 0) (type default))
   )
@@
     (stroke (width 0) (type default))
   )
+  (wire (pts (xy 71.12 34.29) (xy 80.01 34.29))
+    (stroke (width 0) (type default))
+  )
   (wire (pts (xy 31.75 55.88) (xy 34.29 55.88))
     (stroke (width 0) (type default))
@@
     (stroke (width 0) (type default))
   )
-  (wire (pts (xy 52.07 29.21) (xy 77.47 29.21))
-    (stroke (width 0) (type default))
-  )
   (wire (pts (xy 68.58 104.14) (xy 68.58 105.41))
     (stroke (width 0) (type default))
@@
     (stroke (width 0) (type default))
   )
+  (wire (pts (xy 121.92 138.43) (xy 121.92 148.59))
+    (stroke (width 0) (type default))
+  )
   (wire (pts (xy 60.96 173.99) (xy 78.74 173.99))
     (stroke (width 0) (type default))
@@
     (stroke (width 0) (type default))
   )
+  (wire (pts (xy 151.13 148.59) (xy 151.13 166.37))
+    (stroke (width 0) (type default))
+  )
   (wire (pts (xy 43.18 204.47) (xy 43.18 210.82))
     (stroke (width 0) (type default))
@@
     (stroke (width 0) (type default))
   )
-  (wire (pts (xy 80.01 30.48) (xy 80.01 35.56))
+  (wire (pts (xy 80.01 30.48) (xy 80.01 34.29))
     (stroke (width 0) (type default))
   )
@@
   (symbol (lib_id "Connector_Generic:Conn_01x01") (at 59.69 207.01 90) (mirror x) (unit 1)
     (in_bom yes) (on_board yes) (dnp no)
-    (property "Reference" "C" (at 62.23 208.28 90)
+    (property "Reference" "Connector_C" (at 62.23 208.28 90)
       (effects (font (size 1.27 1.27)) (justify right))
     )
-    (property "Value" "Conn_01x01" (at 62.23 205.74 90)
+    (property "Value" "C_connector" (at 62.23 205.74 90)
       (effects (font (size 1.27 1.27)) (justify right))
     )
@@
       (project "neovibe"
         (path "/10e06535-0cd4-4021-8aff-040ddd9278f7"
-          (reference "C") (unit 1)
+          (reference "Connector_C") (unit 1)
         )
       )
@@
     )
   )
+  (symbol (lib_id "power:GND") (at 59.69 39.37 0) (unit 1)
+    (in_bom yes) (on_board yes) (dnp no) (fields_autoplaced)
+    (property "Reference" "#PWR030" (at 59.69 45.72 0)
+      (effects (font (size 1.27 1.27)) hide)
+    )
+    (property "Value" "GND" (at 59.69 44.45 0)
+      (effects (font (size 1.27 1.27)))
+    )
+    (property "Footprint" "" (at 59.69 39.37 0)
+      (effects (font (size 1.27 1.27)) hide)
+    )
+    (property "Datasheet" "" (at 59.69 39.37 0)
+      (effects (font (size 1.27 1.27)) hide)
+    )
+    (pin "1")
+    (instances
+      (project "neovibe"
+        (path "/10e06535-0cd4-4021-8aff-040ddd9278f7"
+          (reference "#PWR030") (unit 1)
+        )
+      )
+    )
+  )
   (symbol (lib_id "Device:Q_NPN_BCE") (at 77.47 40.64 0) (unit 1)
     (in_bom yes) (on_board yes) (dnp no) (fields_autoplaced)
@@
   (symbol (lib_id "Device:C_Polarized") (at 179.07 114.3 90) (unit 1)
     (in_bom yes) (on_board yes) (dnp no) (fields_autoplaced)
-    (property "Reference" "C17" (at 178.181 106.68 90)
+    (property "Reference" "C13" (at 178.181 106.68 90)
       (effects (font (size 1.27 1.27)))
     )
@@
       (project "neovibe"
         (path "/10e06535-0cd4-4021-8aff-040ddd9278f7"
-          (reference "C17") (unit 1)
+          (reference "C13") (unit 1)
         )
       )
@@
   (symbol (lib_id "Device:C_Polarized") (at 241.3 115.57 90) (unit 1)
     (in_bom yes) (on_board yes) (dnp no) (fields_autoplaced)
-    (property "Reference" "C13" (at 240.411 107.95 90)
+    (property "Reference" "C100" (at 240.411 107.95 90)
       (effects (font (size 1.27 1.27)))
     )
@@
       (project "neovibe"
         (path "/10e06535-0cd4-4021-8aff-040ddd9278f7"
-          (reference "C13") (unit 1)
+          (reference "C100") (unit 1)
         )
       )

Commit message: footprints
Parts:
- A1, B1, C16, L1, M1, N1: footprint (none) -> Connector_PinHeader_1.00mm:PinHeader_1x01_P1.00mm_Vertical
- C1, C10, C100, C11, C13, C14, C17, C18, C19, C2, C20, C21, C3, C5, C6, C7, C8: footprint (none) -> Capacitor_THT:CP_Radial_D6.3mm_P2.50mm
- C12: footprint (none) -> Capacitor_THT:C_Rect_L7.2mm_W4.5mm_P5.00mm_FKS2_FKP2_MKS2_MKP2
- C15: footprint (none) -> Capacitor_THT:C_Rect_L7.2mm_W2.5mm_P5.00mm_FKS2_FKP2_MKS2_MKP2
- C22, C23: footprint (none) -> Capacitor_THT:CP_Radial_D5.0mm_P2.50mm
- C24, C25: footprint (none) -> Capacitor_THT:CP_Radial_D12.5mm_P5.00mm
- C26: footprint (none) -> Capacitor_THT:C_Disc_D12.5mm_W5.0mm_P7.50mm
- C4: footprint (none) -> Capacitor_THT:C_Axial_L12.0mm_D6.5mm_P15.00mm_Horizontal
- C9: footprint (none) -> Capacitor_THT:C_Rect_L10.3mm_W5.7mm_P7.50mm_MKS4
- Connector_C1: renamed from Connector_C; footprint (none) -> Connector_PinHeader_1.00mm:PinHeader_1x01_P1.00mm_Vertical
- D1, D2: footprint (none) -> Diode_THT:D_DO-35_SOD27_P3.81mm_Vertical_AnodeUp
- D4: renamed from D; footprint (none) -> Connector_PinHeader_1.00mm:PinHeader_1x01_P1.00mm_Vertical
- E1: renamed from E; footprint (none) -> Connector_PinHeader_1.00mm:PinHeader_1x01_P1.00mm_Vertical
- F1: renamed from F; footprint (none) -> Connector_PinHeader_1.00mm:PinHeader_1x01_P1.00mm_Vertical
- G1: renamed from G; footprint (none) -> Connector_PinHeader_1.00mm:PinHeader_1x01_P1.00mm_Vertical
- H1: renamed from H; footprint (none) -> Connector_PinHeader_1.00mm:PinHeader_1x01_P1.00mm_Vertical
- I1: renamed from I; footprint (none) -> Connector_PinHeader_1.00mm:PinHeader_1x01_P1.00mm_Vertical
- J3: renamed from J; footprint (none) -> Connector_PinHeader_1.00mm:PinHeader_1x01_P1.00mm_Vertical
- K1: renamed from K; footprint (none) -> Connector_PinHeader_1.00mm:PinHeader_1x01_P1.00mm_Vertical
- LA1: footprint (none) -> Connector_PinHeader_1.27mm:PinHeader_1x02_P1.27mm_Vertical
- O1: renamed from O; footprint (none) -> Connector_PinHeader_1.00mm:PinHeader_1x01_P1.00mm_Vertical
- Q1, Q10, Q11, Q12, Q13, Q2, Q3, Q4, Q5, Q6, Q7, Q8, Q9: footprint (none) -> Package_TO_SOT_THT:TO-92L_HandSolder
- R1, R11, R13, R14, R15, R16, R17, R18, R19, R2, R22, R23, R25, R26, R27, R28, R29, R30, R31, R32, R34, R35, R36, R38, R4, R40, R41, R42, R43, R44, R45, R47, R5, R6, R7, R8: footprint (none) -> Resistor_THT:R_Axial_DIN0207_L6.3mm_D2.5mm_P7.62mm_Horizontal
- R10, R12, R20, R21, R24, R3, R33, R37: footprint (none) -> Resistor_THT:R_Axial_DIN0204_L3.6mm_D1.6mm_P5.08mm_Horizontal
- R39, R9: footprint (none) -> Resistor_THT:R_Box_L8.4mm_W2.5mm_P5.08mm
- R46, R49: value R -> 4.7K; footprint (none) -> Resistor_THT:R_Axial_DIN0207_L6.3mm_D2.5mm_P7.62mm_Horizontal
- R48: value R -> 68; footprint (none) -> Resistor_THT:R_Axial_DIN0309_L9.0mm_D3.2mm_P12.70mm_Horizontal
- R50: value R -> 47K; footprint (none) -> Resistor_THT:R_Axial_DIN0204_L3.6mm_D1.6mm_P5.08mm_Horizontal
- RV2: footprint (none) -> Potentiometer_THT:Potentiometer_Vishay_148-149_Single_Vertical
- U1: footprint (none) -> Package_TO_SOT_THT:TO-220-3_Vertical
- X1: renamed from X; footprint (none) -> Connector_PinHeader_1.00mm:PinHeader_1x01_P1.00mm_Vertical
- renumbered RV_Speed to RV_Speed1

Commit message: more placement
Parts:
- renumbered C16 to C101, C100 to C16
Changed lines of the file:
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@@
   (symbol (lib_id "Device:C_Polarized") (at 241.3 115.57 90) (unit 1)
     (in_bom yes) (on_board yes) (dnp no) (fields_autoplaced)
-    (property "Reference" "C100" (at 240.411 107.95 90)
+    (property "Reference" "C16" (at 240.411 107.95 90)
       (effects (font (size 1.27 1.27)))
     )
@@
       (project "neovibe"
         (path "/10e06535-0cd4-4021-8aff-040ddd9278f7"
-          (reference "C100") (unit 1)
+          (reference "C16") (unit 1)
         )
       )
@@
   (symbol (lib_id "Connector_Generic:Conn_01x01") (at 39.37 55.88 0) (unit 1)
     (in_bom yes) (on_board yes) (dnp no) (fields_autoplaced)
-    (property "Reference" "C16" (at 41.91 54.61 0)
+    (property "Reference" "C101" (at 41.91 54.61 0)
       (effects (font (size 1.27 1.27)) (justify left))
     )
@@
       (project "neovibe"
         (path "/10e06535-0cd4-4021-8aff-040ddd9278f7"
-          (reference "C16") (unit 1)
+          (reference "C101") (unit 1)
         )
       )
